File: ai03-pcb-guide.kicad_pcb (KiCad board)
At the start: 2 copper layers, 24 parts, among them SW1 SW_Push, U1 ATmega32U4-AU, Y1 Crystal_GND24_Small

Commit message: PCB changes
Parts:
- C1, C2, C3, C4, C5, C6, C7, D1, D2, D3, D4, F1, R1, R2, R3, R4, SW1, U1, USB1, Y1: moved to B.Cu
- moved R2 86.2 mm to (92.1, 127.0), turned to 270 degrees
- moved R3 81.3 mm to (88.9, 127.0), turned to 270 degrees
- moved USB1 80.9 mm to (90.9, 116.3), turned to 270 degrees
- moved F1 73.8 mm to (84.9, 130.2), turned to 90 degrees
- moved C1 72.9 mm to (110.7, 124.0), turned to 270 degrees
- moved R4 70.0 mm to (99.8, 124.5), turned to 90 degrees
- moved C5 63.3 mm to (103.0, 124.5), turned to 90 degrees
- moved SW1 63.3 mm to (91.3, 146.8), turned to 180 degrees
- moved C2 60.3 mm to (118.5, 124.1), turned to 90 degrees
- moved R1 60.3 mm to (104.0, 131.0), turned to 270 degrees
- moved C3 59.7 mm to (103.2, 134.9), turned to 180 degrees
- moved C7 57.3 mm to (110.0, 145.1)
- moved Y1 54.9 mm to (114.5, 124.1)
- moved MX2 53.5 mm to (153.9, 124.0)
- moved C4 51.1 mm to (122.9, 132.0), turned to 90 degrees
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Routing:
- net GND: track 0.00 -> 48.6 mm
- net Net-(R3-Pad2): track 0.00 -> 29.4 mm
- net Net-(R2-Pad2): track 0.00 -> 25.0 mm
- net VCC: track 0.00 -> 9.77 mm
- net D+: track 0.00 -> 5.76 mm
- net D-: track 0.00 -> 5.75 mm
- net Net-(C2-Pad1): track 0.00 -> 2.87 mm
- net Net-(C1-Pad1): track 0.00 -> 2.80 mm
Other:
- board outline added: 81.8 x 38.1 mm
- net class Default: trace_width 0.25 -> 0.254
- net class Power added: clearance 0.2, trace_width 0.381, via_dia 0.8, via_drill 0.4

Commit message: Kicad edits
Parts:
- moved R4 28.4 mm to (123.1, 140.7), turned to 270 degrees
- moved C2 9.17 mm to (109.3, 125.1), turned to 270 degrees
- moved C1 6.51 mm to (117.1, 125.3), turned to 90 degrees
- moved C5 4.08 mm to (104.1, 128.4)
- moved R1 3.96 mm to (101.0, 128.4), turned to 90 degrees
- moved C3 1.68 mm to (104.6, 134.1)
- moved Y1 1.60 mm to (113.3, 125.1), turned to 180 degrees
Routing:
- net GND: track 48.6 -> 71.0 mm
- net Net-(R1-Pad1): track 0.00 -> 21.8 mm, vias 0 -> 3
- net +5V: track 0.00 -> 10.9 mm
- net Net-(C2-Pad1): track 2.87 -> 10.9 mm
- net Net-(C1-Pad1): track 2.80 -> 7.19 mm
- net Net-(C3-Pad1): track 0.00 -> 3.69 mm
- net Net-(R4-Pad1): track 0.00 -> 3.08 mm

Commit message: PCB completed
Parts:
- moved C7 6.65 mm to (104.3, 141.6), turned to 270 degrees
- moved C3 2.93 mm to (101.7, 134.4)
- moved C1 2.38 mm to (117.1, 122.9)
- moved C2 2.38 mm to (109.3, 122.7)
- moved Y1 2.38 mm to (113.3, 122.7)
Routing:
- net +5V: track 10.9 -> 117.6 mm, vias 0 -> 5
- net GND: track 71.0 -> 154.5 mm
- net ROW1: track 0.00 -> 50.5 mm
- net COL1: track 0.00 -> 50.2 mm
- net ROW0: track 0.00 -> 47.3 mm
- net COL0: track 0.00 -> 30.8 mm
- net Net-(R1-Pad1): track 21.8 -> 33.8 mm, vias 3 -> 2
- net Net-(D1-Pad2): track 0.00 -> 7.38 mm
- net Net-(D4-Pad2): track 0.00 -> 7.36 mm
- net Net-(D2-Pad2): track 0.00 -> 7.36 mm
- net Net-(D3-Pad2): track 0.00 -> 7.23 mm
- net Net-(C3-Pad1): track 3.69 -> 6.50 mm
- net Net-(C1-Pad1): track 7.19 -> 9.57 mm
- net Net-(C2-Pad1): track 10.9 -> 13.3 mm

Commit message: PCB Design complete
Routing:
- net Net-(USB1-Pad6): track 0.00 -> 16.3 mm
- net Net-(D4-Pad2): track 7.36 -> 7.95 mm
- net Net-(D3-Pad2): track 7.23 -> 7.83 mm
- net Net-(D2-Pad2): track 7.36 -> 7.95 mm
- net Net-(D1-Pad2): track 7.38 -> 7.98 mm
- added copper zone on B.Cu, net GND
Other:
- board text added: "PizzaPad1"
Changed lines of the file:
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@@
   (general
     (thickness 1.6)
-    (drawings 8)
-    (tracks 202)
+    (drawings 9)
+    (tracks 213)
     (zones 0)
     (modules 24)
@@
     (34 B.Paste user)
     (35 F.Paste user)
-    (36 B.SilkS user hide)
+    (36 B.SilkS user)
     (37 F.SilkS user)
     (38 B.Mask user)
@@
     (46 B.CrtYd user)
     (47 F.CrtYd user)
-    (48 B.Fab user hide)
+    (48 B.Fab user)
     (49 F.Fab user)
   )
@@
     (visible_elements 7FFFFFFF)
     (pcbplotparams
-      (layerselection 0x010fc_ffffffff)
-      (usegerberextensions false)
+      (layerselection 0x010f0_ffffffff)
+      (usegerberextensions true)
       (usegerberattributes false)
       (usegerberadvancedattributes false)
@@
       (plotinvisibletext false)
       (padsonsilk false)
-      (subtractmaskfromsilk false)
+      (subtractmaskfromsilk true)
       (outputformat 1)
       (mirror false)
-      (drillshape 1)
+      (drillshape 0)
       (scaleselection 1)
-      (outputdirectory ""))
+      (outputdirectory "Gerbers/"))
   )
   (net 0 "")
@@
       (rotate (xyz 0 0 0))
     )
+  )
+  (gr_text PizzaPad1 (at 115.09375 115.8875) (layer F.SilkS)
+    (effects (font (size 1 1) (thickness 0.15)))
   )
   (gr_line (start 81.75625 116.68125) (end 81.75625 150.01875) (layer Edge.Cuts) (width 0.05))
@@
   (segment (start 142.875 122.302) (end 142.875 121.44375) (width 0.254) (layer B.Cu) (net 6))
   (segment (start 142.875 121.44375) (end 140.30325 118.872) (width 0.254) (layer B.Cu) (net 6))
+  (segment (start 137.374 118.912) (end 137.414 118.872) (width 0.254) (layer B.Cu) (net 6))
+  (segment (start 137.374 119.452) (end 137.374 118.912) (width 0.254) (layer B.Cu) (net 6))
   (segment (start 143.025 125.602) (end 144.423 127) (width 0.254) (layer B.Cu) (net 7))
   (segment (start 142.875 125.602) (end 143.025 125.602) (width 0.254) (layer B.Cu) (net 7))
@@
   (segment (start 161.8615 122.302) (end 161.8615 121.38025) (width 0.254) (layer B.Cu) (net 8))
   (segment (start 161.8615 121.38025) (end 159.35325 118.872) (width 0.254) (layer B.Cu) (net 8))
+  (segment (start 156.424 118.912) (end 156.464 118.872) (width 0.254) (layer B.Cu) (net 8))
+  (segment (start 156.424 119.452) (end 156.424 118.912) (width 0.254) (layer B.Cu) (net 8))
   (segment (start 140.0855 137.922) (end 137.414 137.922) (width 0.254) (layer B.Cu) (net 9))
   (segment (start 142.8115 141.352) (end 142.8115 140.648) (width 0.254) (layer B.Cu) (net 9))
   (segment (start 142.8115 140.648) (end 140.0855 137.922) (width 0.254) (layer B.Cu) (net 9))
+  (segment (start 137.374 137.962) (end 137.414 137.922) (width 0.254) (layer B.Cu) (net 9))
+  (segment (start 137.374 138.502) (end 137.374 137.962) (width 0.254) (layer B.Cu) (net 9))
   (segment (start 161.7115 144.652) (end 160.3135 146.05) (width 0.254) (layer B.Cu) (net 10))
   (segment (start 161.8615 144.652) (end 161.7115 144.652) (width 0.254) (layer B.Cu) (net 10))
@@
   (segment (start 161.8615 141.352) (end 161.8615 140.43025) (width 0.254) (layer B.Cu) (net 11))
   (segment (start 161.8615 140.43025) (end 159.35325 137.922) (width 0.254) (layer B.Cu) (net 11))
+  (segment (start 156.424 137.962) (end 156.464 137.922) (width 0.254) (layer B.Cu) (net 11))
+  (segment (start 156.424 138.502) (end 156.424 137.962) (width 0.254) (layer B.Cu) (net 11))
   (segment (start 84.93125 128.05) (end 84.93125 128.775) (width 0.254) (layer B.Cu) (net 12))
   (segment (start 84.93125 126.5165) (end 84.93125 128.05) (width 0.254) (layer B.Cu) (net 12))
@@
   (segment (start 120.04725 139.7785) (end 120 139.73125) (width 0.254) (layer B.Cu) (net 20))
   (segment (start 123.063 139.7785) (end 120.04725 139.7785) (width 0.254) (layer B.Cu) (net 20))
+  (segment (start 87.2185 120.80025) (end 87.2185 116.30025) (width 0.254) (layer B.Cu) (net 43))
+  (segment (start 87.2185 116.30025) (end 94.5185 116.30025) (width 0.254) (layer B.Cu) (net 43))
+  (segment (start 94.5185 120.80025) (end 94.5185 116.30025) (width 0.254) (layer B.Cu) (net 43))
+  (zone (net 1) (net_name GND) (layer B.Cu) (hatch edge 0.508)
+    (connect_pads (clearance 0.508))
+    (min_thickness 0.254)
+    (fill yes (arc_segments 32) (thermal_gap 0.508) (thermal_bridge_width 0.508))
+    (polygon
+      (pts
+        (xy 109.5375 130.96875) (xy 119.0625 130.96875) (xy 119.0625 140.49375) (xy 109.5375 140.49375)
+      )
+    )
+  )
+  (zone (net 1) (net_name GND) (layer B.Cu) (hatch edge 0.508)
+    (connect_pads (clearance 0.508))
+    (min_thickness 0.254)
+    (fill yes (arc_segments 32) (thermal_gap 0.508) (thermal_bridge_width 0.508))
+    (polygon
+      (pts
+        (xy 121.44375 127.79375) (xy 104.775 127.79375) (xy 104.775 119.0625) (xy 121.44375 119.0625)
+      )
+    )
+  )
+  (zone (net 1) (net_name GND) (layer B.Cu) (hatch edge 0.508)
+    (connect_pads (clearance 0.508))
+    (min_thickness 0.254)
+    (fill yes (arc_segments 32) (thermal_gap 0.508) (thermal_bridge_width 0.508))
+    (polygon
+      (pts
+        (xy 85.725 115.09375) (xy 96.04375 115.09375) (xy 96.04375 122.2375) (xy 85.725 122.2375)
+      )
+    )
+  )
 )
